File: hardware/aquarium-control.sch (KiCad schematic (older format))
At the start: 0 parts

Commit message: Desgined power regulation circuitry
Parts:
- added C?: 220u, symbol CP1
- added C?: 22u, symbol CP1
- added D?: DIODESCH, symbol DIODESCH
- added L?: INDUCTOR, symbol INDUCTOR
- added U1: LM2574N, symbol LM2574N
- added U2, U3: D3043, symbol D3043
Connections:
- new net: C?.1, L?.2, U1.1 (FB)
- new net: D?.2 (K), L?.1, U1.7 (Out)
- new net +12V: C?.1, U1.5 (Vin)
- new net GND: C?.2, C?.2, D?.1 (A), U1.2 (GND), U1.3 (OFF), U1.4 (GND)
Changed lines of the file:
@@
-EESchema Schematic File Version 2  date Mon 06 May 2013 08:58:37 PM PDT
+EESchema Schematic File Version 2  date Mon 06 May 2013 11:24:16 PM PDT
 LIBS:power
 LIBS:device
@@
 LIBS:contrib
 LIBS:valves
-EELAYER 43  0
+LIBS:aquarium-control-cache
+EELAYER 25  0
 EELAYER END
 $Descr A4 11700 8267
@@
 Comment4 ""
 $EndDescr
+Connection ~ 3800 4600
+Wire Wire Line
+	3800 4000 3800 4600
+Wire Wire Line
+	3800 4600 3800 4700
+Wire Wire Line
+	4400 4400 4200 4400
+Wire Wire Line
+	4200 4400 3650 4400
+Wire Wire Line
+	5200 4900 5200 5000
+Wire Wire Line
+	5200 4500 5200 4400
+Wire Wire Line
+	5200 4400 5200 4100
+Connection ~ 5200 4400
+Wire Wire Line
+	5200 4100 2400 4100
+Wire Wire Line
+	2400 4100 2400 4300
+Wire Wire Line
+	2400 4300 2500 4300
+Wire Wire Line
+	3800 5100 3800 5200
+Connection ~ 2300 4500
+Wire Wire Line
+	2300 4800 2300 4600
+Wire Wire Line
+	2300 4600 2300 4500
+Wire Wire Line
+	2300 4500 2300 4400
+Wire Wire Line
+	2300 4400 2500 4400
+Wire Wire Line
+	2300 4600 2500 4600
+Wire Wire Line
+	2300 4500 2500 4500
+Connection ~ 2300 4600
+Wire Wire Line
+	3800 4600 3650 4600
+Wire Wire Line
+	4200 4400 4200 4500
+Connection ~ 4200 4400
+Wire Wire Line
+	4200 4900 4200 5000
+Wire Wire Line
+	5000 4400 5200 4400
+$Comp
+L +12V #PWR?
+U 1 1 51889D9C
+P 3800 4000
+F 0 "#PWR?" H 3800 3950 20  0001 C CNN
+F 1 "+12V" H 3800 4100 30  0000 C CNN
+	1    3800 4000
+	1    0    0    -1
+$EndComp
+$Comp
+L GND #PWR?
+U 1 1 51889CEB
+P 5200 5000
+F 0 "#PWR?" H 5200 5000 30  0001 C CNN
+F 1 "GND" H 5200 4930 30  0001 C CNN
+	1    5200 5000
+	1    0    0    -1
+$EndComp
+$Comp
+L GND #PWR?
+U 1 1 51889CE8
+P 4200 5000
+F 0 "#PWR?" H 4200 5000 30  0001 C CNN
+F 1 "GND" H 4200 4930 30  0001 C CNN
+	1    4200 5000
+	1    0    0    -1
+$EndComp
+$Comp
+L GND #PWR?
+U 1 1 51889C59
+P 3800 5200
+F 0 "#PWR?" H 3800 5200 30  0001 C CNN
+F 1 "GND" H 3800 5130 30  0001 C CNN
+	1    3800 5200
+	1    0    0    -1
+$EndComp
+$Comp
+L GND #PWR?
+U 1 1 51889C28
+P 2300 4800
+F 0 "#PWR?" H 2300 4800 30  0001 C CNN
+F 1 "GND" H 2300 4730 30  0001 C CNN
+	1    2300 4800
+	1    0    0    -1
+$EndComp
+$Comp
+L DIODESCH D?
+U 1 1 51889BF9
+P 4200 4700
+F 0 "D?" H 4200 4800 40  0000 C CNN
+F 1 "DIODESCH" H 4200 4600 40  0000 C CNN
+	1    4200 4700
+	0    -1   -1   0
+$EndComp
+$Comp
+L INDUCTOR L?
+U 1 1 51889BDF
+P 4700 4400
+F 0 "L?" V 4650 4400 40  0000 C CNN
+F 1 "INDUCTOR" V 4800 4400 40  0000 C CNN
+	1    4700 4400
+	0    -1   -1   0
+$EndComp
+$Comp
+L CP1 C?
+U 1 1 51889BB6
+P 3800 4900
+F 0 "C?" H 3850 5000 50  0000 L CNN
+F 1 "22u" H 3850 4800 50  0000 L CNN
+	1    3800 4900
+	1    0    0    -1
+$EndComp
+$Comp
+L CP1 C?
+U 1 1 51889BAC
+P 5200 4700
+F 0 "C?" H 5250 4800 50  0000 L CNN
+F 1 "220u" H 5250 4600 50  0000 L CNN
+	1    5200 4700
+	1    0    0    -1
+$EndComp
+$Comp
+L LM2574N U1
+U 1 1 51889B56
+P 3050 4550
+F 0 "U1" H 3300 4600 60  0000 C CNN
+F 1 "LM2574N" H 2950 4600 60  0000 C CNN
+	1    3050 4550
+	0    1    1    0
+$EndComp
+$Comp
+L D3043 U3
+U 1 1 518899F6
+P 7550 3950
+F 0 "U3" H 7050 3950 60  0000 C CNN
+F 1 "D3043" H 7450 3950 60  0000 C CNN
+	1    7550 3950
+	1    0    0    -1
+$EndComp
+$Comp
+L D3043 U2
+U 1 1 518899F2
+P 6650 3950
+F 0 "U2" H 6150 3950 60  0000 C CNN
+F 1 "D3043" H 6550 3950 60  0000 C CNN
+	1    6650 3950
+	1    0    0    -1
+$EndComp
 $EndSCHEMATC

Commit message: Finished the hardware schematic
Parts:
- added P1: CONN_4, symbol CONN_4
- added P2, P3: CONN_2, symbol CONN_2
- added U2: CD40109B, symbol CD40109B
- gave numbers to parts that had none: 4
- renumbered U2 to U3, U3 to U4
Connections:
- net +12V: now also U3.3, U4.3
- net GND: now also P2.2 (PM), P3.2 (PM), U2.8 (VSS)
- net at U3.1: now also U2.4 (E)
- net at U3.10: now also U2.5 (F)
- net at U3.2: now also P2.1 (P1)
- net at U4.1: now also U2.11 (G)
- net at U4.10: now also U2.13 (H)
- net at U4.2: now also P3.1 (P1)
- net at C2.1, L1.2, U1.1 (FB): now also U2.16 (VDD)
- new net: P1.3 (P3), U2.10 (C)
- new net: P1.4 (P4), U2.14 (D)
- new net: P1.1 (P1), U2.3 (A)
- new net: P1.2 (P2), U2.6 (B)
- new net +3.3V: U2.1 (VCC), U2.15 (END), U2.2 (ENA), U2.7 (ENB), U2.9 (ENC)
Other:
- moved on the sheet: U3, U4

Commit message: Finished the first draft of the board
Parts:
- removed P1: CONN_4, symbol CONN_4
- added D2: Night LED, symbol LED
- added D3: Day LED, symbol LED
- added D4: Control LED, symbol LED
- added F? (x2): FUSE, symbol FUSE
- added P1: R.Pi, symbol CONN_3X2
- added P4: Power, symbol CONN_2
- added P5: Switch, symbol CONN_3
- added RP?: R_PACK4, symbol R_PACK4
- P2: value CONN_2 -> Day
- P3: value CONN_2 -> Night
Connections:
- net +12V: now also D4.1 (A), P5.1 (P1)
- net GND: now also P1.6, P4.2 (PM), RP?.1 (P1), RP?.2 (P2), RP?.3 (P3)
- net at P2.1 (P1), U3.2: now also D3.1 (A), P5.3 (P3)
- net at P3.1 (P1), U4.2: now also D2.1 (A)
- net at U2.10 (C): now also P1.4
- net at U2.14 (D): now also P1.5
- net at U2.3 (A): now also P1.2
- net at U2.6 (B): now also P1.3
- net +3.3V: no longer names the net of U2.1 (VCC), U2.15 (END), U2.2 (ENA), U2.7 (ENB), U2.9 (ENC)
- net +3.3V: now also F?.2
- new net: F?.1, P1.1
- new net: F?.1, P4.1 (P1)
- new net: F?.2, P5.2 (PM)
- new net: D4.2 (K), RP?.6 (R3)
- new net: D3.2 (K), RP?.7 (R2)
- new net: D2.2 (K), RP?.8 (R1)
Other:
- moved on the sheet: C1, C2, D1, L1, P2, P3, U1

Commit message: Named all components and generated the netlist
Parts:
- gave numbers to parts that had none: 3
Changed lines of the file:
@@
-EESchema Schematic File Version 2  date Tue 07 May 2013 09:58:51 PM PDT
+EESchema Schematic File Version 2  date Wed 08 May 2013 09:01:33 PM PDT
 LIBS:power
 LIBS:device
@@
 Sheet 1 1
 Title ""
-Date "8 may 2013"
+Date "9 may 2013"
 Rev ""
 Comp ""
@@
 	9000 2400 9000 2500
 $Comp
-L +12V #PWR?
+L +12V #PWR01
 U 1 1 5189DA8F
 P 9800 2300
-F 0 "#PWR?" H 9800 2250 20  0001 C CNN
+F 0 "#PWR01" H 9800 2250 20  0001 C CNN
 F 1 "+12V" H 9800 2400 30  0000 C CNN
 	1    9800 2300
@@
 $EndComp
 $Comp
-L GND #PWR?
+L GND #PWR02
 U 1 1 5189D921
 P 9400 3700
-F 0 "#PWR?" H 9400 3700 30  0001 C CNN
+F 0 "#PWR02" H 9400 3700 30  0001 C CNN
 F 1 "GND" H 9400 3630 30  0001 C CNN
 	1    9400 3700
@@
 $EndComp
 $Comp
-L R_PACK4 RP?
+L R_PACK4 RP1
 U 1 1 5189D8A9
 P 9650 3300
-F 0 "RP?" H 9650 3750 40  0000 C CNN
+F 0 "RP1" H 9650 3750 40  0000 C CNN
 F 1 "R_PACK4" H 9650 3250 40  0000 C CNN
 	1    9650 3300
@@
 $EndComp
 $Comp
-L GND #PWR?
+L GND #PWR03
 U 1 1 5189D42C
 P 8750 4300
-F 0 "#PWR?" H 8750 4300 30  0001 C CNN
+F 0 "#PWR03" H 8750 4300 30  0001 C CNN
 F 1 "GND" H 8750 4230 30  0001 C CNN
 	1    8750 4300
@@
 $EndComp
 $Comp
-L +12V #PWR?
+L +12V #PWR04
 U 1 1 5189D3FC
 P 8750 4700
-F 0 "#PWR?" H 8750 4650 20  0001 C CNN
+F 0 "#PWR04" H 8750 4650 20  0001 C CNN
 F 1 "+12V" H 8750 4800 30  0000 C CNN
 	1    8750 4700
@@
 $EndComp
 $Comp
-L FUSE F?
+L FUSE F2
 U 1 1 5189C531
 P 8550 4450
-F 0 "F?" H 8650 4500 40  0000 C CNN
+F 0 "F2" H 8650 4500 40  0000 C CNN
 F 1 "FUSE" H 8450 4400 40  0000 C CNN
 	1    8550 4450
@@
 $EndComp
 $Comp
-L FUSE F?
+L FUSE F1
 U 1 1 5189C52A
 P 4350 2500
-F 0 "F?" H 4450 2550 40  0000 C CNN
+F 0 "F1" H 4450 2550 40  0000 C CNN
 F 1 "FUSE" H 4250 2450 40  0000 C CNN
 	1    4350 2500
@@
 $EndComp
 $Comp
-L GND #PWR?
+L GND #PWR05
 U 1 1 5189C3E5
 P 4900 3500
-F 0 "#PWR?" H 4900 3500 30  0001 C CNN
+F 0 "#PWR05" H 4900 3500 30  0001 C CNN
 F 1 "GND" H 4900 3430 30  0001 C CNN
 	1    4900 3500
@@
 $EndComp
 $Comp
-L GND #PWR?
+L GND #PWR06
 U 1 1 5188A4BE
 P 8100 3500
-F 0 "#PWR?" H 8100 3500 30  0001 C CNN
+F 0 "#PWR06" H 8100 3500 30  0001 C CNN
 F 1 "GND" H 8100 3430 30  0001 C CNN
 	1    8100 3500
@@
 $EndComp
 $Comp
-L GND #PWR?
+L GND #PWR07
 U 1 1 5188A4B9
 P 8100 2300
-F 0 "#PWR?" H 8100 2300 30  0001 C CNN
+F 0 "#PWR07" H 8100 2300 30  0001 C CNN
 F 1 "GND" H 8100 2230 30  0001 C CNN
 	1    8100 2300
@@
 $EndComp
 $Comp
-L +12V #PWR?
+L +12V #PWR08
 U 1 1 5188A4A6
 P 8000 3100
-F 0 "#PWR?" H 8000 3050 20  0001 C CNN
+F 0 "#PWR08" H 8000 3050 20  0001 C CNN
 F 1 "+12V" H 8000 3200 30  0000 C CNN
 	1    8000 3100
@@
 $EndComp
 $Comp
-L +12V #PWR?
+L +12V #PWR09
 U 1 1 5188A46D
 P 7600 1900
-F 0 "#PWR?" H 7600 1850 20  0001 C CNN
+F 0 "#PWR09" H 7600 1850 20  0001 C CNN
 F 1 "+12V" H 7600 2000 30  0000 C CNN
 	1    7600 1900
@@
 $EndComp
 $Comp
-L GND #PWR?
+L GND #PWR010
 U 1 1 5188A2B0
 P 5200 3600
-F 0 "#PWR?" H 5200 3600 30  0001 C CNN
+F 0 "#PWR010" H 5200 3600 30  0001 C CNN
 F 1 "GND" H 5200 3530 30  0001 C CNN
 	1    5200 3600
@@
 $EndComp
 $Comp
-L +12V #PWR?
+L +12V #PWR011
 U 1 1 51889D9C
 P 5300 3900
-F 0 "#PWR?" H 5300 3850 20  0001 C CNN
+F 0 "#PWR011" H 5300 3850 20  0001 C CNN
 F 1 "+12V" H 5300 4000 30  0000 C CNN
 	1    5300 3900
@@
 $EndComp
 $Comp
-L GND #PWR?
+L GND #PWR012
 U 1 1 51889CEB
 P 6700 4600
-F 0 "#PWR?" H 6700 4600 30  0001 C CNN
+F 0 "#PWR012" H 6700 4600 30  0001 C CNN
 F 1 "GND" H 6700 4530 30  0001 C CNN
 	1    6700 4600
@@
 $EndComp
 $Comp
-L GND #PWR?
+L GND #PWR013
 U 1 1 51889CE8
 P 5700 4600
-F 0 "#PWR?" H 5700 4600 30  0001 C CNN
+F 0 "#PWR013" H 5700 4600 30  0001 C CNN
 F 1 "GND" H 5700 4530 30  0001 C CNN
 	1    5700 4600
@@
 $EndComp
 $Comp
-L GND #PWR?
+L GND #PWR014
 U 1 1 51889C59
 P 5300 4800
-F 0 "#PWR?" H 5300 4800 30  0001 C CNN
+F 0 "#PWR014" H 5300 4800 30  0001 C CNN
 F 1 "GND" H 5300 4730 30  0001 C CNN
 	1    5300 4800
@@
 $EndComp
 $Comp
-L GND #PWR?
+L GND #PWR015
 U 1 1 51889C28
 P 3900 4400
-F 0 "#PWR?" H 3900 4400 30  0001 C CNN
+F 0 "#PWR015" H 3900 4400 30  0001 C CNN
 F 1 "GND" H 3900 4330 30  0001 C CNN
 	1    3900 4400

Commit message: Fixed the LED footprint
Changed lines of the file:
@@
-EESchema Schematic File Version 2  date Wed 08 May 2013 09:01:33 PM PDT
+EESchema Schematic File Version 2  date Thu 09 May 2013 08:46:26 AM PDT
 LIBS:power
 LIBS:device
@@
 	9400 2500 9400 1800
 Wire Wire Line
-	9400 1800 8300 1800
+	8300 1800 9400 1800
 Wire Wire Line
 	9800 2500 9800 2300
 Connection ~ 9400 3600
 Wire Wire Line
-	9400 3500 9400 3600
-Wire Wire Line
-	9400 3600 9400 3700
+	9400 3500 9400 3700
 Wire Wire Line
 	9400 3100 9400 2900
 Wire Wire Line
-	8300 1800 8300 2000
-Wire Wire Line
-	8300 2000 8300 5000
+	8300 1800 8300 5000
 Wire Wire Line
 	9300 3100 9300 3000
@@
 	8750 4200 8850 4200
 Wire Wire Line
-	8500 3200 8400 3200
-Wire Wire Line
-	8400 3200 7500 3200
+	8500 3200 7500 3200
 Wire Wire Line
 	8850 4900 8550 4900
@@
 	8550 4900 8550 4700
 Wire Wire Line
-	8500 2000 8300 2000
-Wire Wire Line
-	8300 2000 7500 2000
+	8500 2000 7500 2000
 Wire Wire Line
 	3800 2500 3800 3100
@@
 Connection ~ 5200 2500
 Wire Wire Line
-	4600 2500 5200 2500
-Wire Wire Line
-	5200 2500 6800 2500
+	6800 2500 4600 2500
 Wire Wire Line
 	3800 3100 4000 3100
@@
 Connection ~ 6800 2900
 Wire Wire Line
-	6600 3000 6800 3000
+	6800 3000 6600 3000
 Wire Wire Line
 	7400 3100 7400 3200
@@
 Connection ~ 5200 2900
 Wire Wire Line
-	5300 3000 5200 3000
+	5200 3000 5300 3000
 Wire Wire Line
 	5700 4500 5700 4600
@@
 	3900 4200 4000 4200
 Wire Wire Line
-	4000 4000 3900 4000
-Wire Wire Line
-	3900 4000 3900 4100
-Wire Wire Line
-	3900 4100 3900 4200
-Wire Wire Line
-	3900 4200 3900 4400
+	3900 4000 4000 4000
+Wire Wire Line
+	3900 4400 3900 4000
 Connection ~ 3900 4100
 Wire Wire Line
@@
 	6700 4500 6700 4600
 Wire Wire Line
-	5900 4000 5700 4000
-Wire Wire Line
-	5700 4000 5150 4000
-Wire Wire Line
-	5300 3900 5300 4200
-Wire Wire Line
-	5300 4200 5300 4300
+	5900 4000 5150 4000
+Wire Wire Line
+	5300 3900 5300 4300
 Connection ~ 5300 4200
 Wire Wire Line
@@
 	6700 4000 6500 4000
 Wire Wire Line
-	6600 2800 6700 2800
+	6700 2800 6600 2800
 Wire Wire Line
 	6600 3100 7100 3100
@@
 	4900 3300 4900 3500
 Wire Wire Line
-	5200 3000 5200 2900
-Wire Wire Line
-	5200 2900 5200 2800
-Wire Wire Line
-	5200 2800 5200 2500
-Wire Wire Line
-	6800 3000 6800 2900
-Wire Wire Line
-	6800 2900 6800 2500
+	5200 2500 5200 3000
+Wire Wire Line
+	6800 2500 6800 3000
 Wire Wire Line
 	5300 2800 5200 2800
 Wire Wire Line
-	6700 2800 6700 3700
-Wire Wire Line
-	6700 3700 6700 4000
-Wire Wire Line
-	6700 4000 6700 4100
+	6700 4100 6700 2800
 Connection ~ 6700 3700
 Wire Wire Line
@@
 Connection ~ 8400 3200
 Wire Wire Line
-	9300 3500 9300 3600
-Wire Wire Line
-	9500 3500 9500 3600
-Wire Wire Line
-	9500 3600 9400 3600
-Wire Wire Line
-	9400 3600 9300 3600
+	9300 3600 9300 3500
+Wire Wire Line
+	9500 3600 9500 3500
+Wire Wire Line
+	9300 3600 9500 3600
 Wire Wire Line
 	8400 3200 8400 2400
