File: hardware/aquarium-control.sch (KiCad schematic (older format))
At the start: 31 parts, among them M1 CONN_1, M2 CONN_1, P1 Raspberry Pi, P2 Day, P3 Night, P4 Power, P5 Switch, U1 SN74HC04, U2 MDC3105D, U3 IM03GR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

Commit message: Version 2.5 of the hardware designed.
Parts:
- L1: value INDUCTOR -> 47u
Changed lines of the file:
@@
-EESchema Schematic File Version 2  date 7/9/2013 11:11:05 PM
+EESchema Schematic File Version 2  date 7/9/2013 11:29:03 PM
 LIBS:power
 LIBS:device
@@
 P 8200 1200
 F 0 "L1" V 8150 1200 40  0000 C CNN
-F 1 "INDUCTOR" V 8300 1200 40  0000 C CNN
+F 1 "47u" V 8300 1200 40  0000 C CNN
 F 2 "~" H 8200 1200 60  0000 C CNN
 F 3 "~" H 8200 1200 60  0000 C CNN
