File: board/Aquarium Control.kicad_pcb (KiCad board)
At the start: 2 copper layers, 16 x 57 mm, 8 parts, among them J2 CONN_04SCREW, J3 Raspberry_Pi_2_3, U1 10118194-MICRO-USB, U2 10118194-MICRO-USB, U3 SN74LVC1T45DBVRDBV6-M, U4 SN74LVC1T45DBVRDBV6-M

Commit message: New board revision
Parts:
- added J1: Conn_01x02_Pin, Connector_PinHeader_2.54mm:PinHeader_1x02_P2.54mm_Vertical, F.Cu at (145.7, 64.0)
- moved J3 2.14 mm to (146.0, 68.9)
Routing:
- net GND: track 83.7 -> 93.8 mm
- net +5V: track 56.7 -> 62.3 mm
- net +3.3V: track 31.8 -> 28.8 mm
- net Net-(J3-MOSI0/GPIO10): track 20.4 -> 18.2 mm
- net Net-(J3-SCLK0/GPIO11): track 22.8 -> 20.6 mm
Other:
- board text added: "Aquarium Control v3.1 Copyright Bryan Hughes November 2025"
- board text removed: "Aquarium Control v3.0 Copyright Bryan Hughes November 2025"
