File: board/Aquarium Control.kicad_sch (KiCad schematic)
At the start: 8 parts, among them J2 CONN_04SCREW, J3 Raspberry_Pi_2_3, U1 10118194-MICRO-USB, U2 10118194-MICRO-USB, U3 SN74LVC1T45DBVRDBV6-M, U4 SN74LVC1T45DBVRDBV6-M

Commit message: New board revision
Parts:
- added J1: Conn_01x02_Pin, Connector_PinHeader_2.54mm:PinHeader_1x02_P2.54mm_Vertical, symbol Connector:Conn_01x02_Pin
Connections:
- net +5V: now also J1.1 (Pin_1)
- net GND: now also J1.2 (Pin_2)
